File: ecse-2023-project.kicad_sch (KiCad schematic)
At the start: 13 parts, among them J1 Barrel_Jack, J2 Screw_Terminal_01x02, J3 Screw_Terminal_01x02, J4 Screw_Terminal_01x03, J5 Conn_01x03_Female, J6 Conn_02x02_Counter_Clockwise, J7 Conn_01x02_Pin, Q1 IRF740, Q2 IRF740, U1 ESP32_DevKit_V1_DOIT

Commit message: Q1/Q2 are IRLZ44N, not IRF740
The fitted parts are IRLZ44N. The IRF740 value was wrong in a way that
matters: its gate threshold is around 4V, so a 3.3V ESP32 GPIO would never
fully turn it on and it would run hot in partial conduction. The IRLZ44N is
logic-level and switches fully from 3.3V drive.

Both symbols extend BUZ11, so the pinout and TO-220 footprint are unchanged.
Parts:
- Q1, Q2: value IRF740 -> IRLZ44N; symbol Transistor_FET:IRF740 -> Transistor_FET:IRLZ44N
Changed lines of the file:
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@@
 	)
 	(symbol
-		(lib_id "Transistor_FET:IRF740")
+		(lib_id "Transistor_FET:IRLZ44N")
 		(at 175.26 97.79 90)
 		(unit 1)
@@
 			)
 		)
-		(property "Value" "IRF740"
+		(property "Value" "IRLZ44N"
 			(at 175.26 90.17 90)
 			(effects
@@
 	)
 	(symbol
-		(lib_id "Transistor_FET:IRF740")
+		(lib_id "Transistor_FET:IRLZ44N")
 		(at 156.21 97.79 90)
 		(unit 1)
@@
 			)
 		)
-		(property "Value" "IRF740"
+		(property "Value" "IRLZ44N"
 			(at 156.21 90.17 90)
 			(effects
